Commit message: add milestone 2

File: urdf/real_steel.urdf (robot description, URDF)
Before this commit: robot real_steel, 9 links, 8 joints
Links:
- added link l_shoulder_roll_link, mass 0.02; collision sphere radius=0.025; visual sphere radius=0.025
- added link r_shoulder_roll_link, mass 0.02; collision sphere radius=0.025; visual sphere radius=0.025
- link l_shoulder_pan_link: mass 0.02 -> 0.1; geometry collision cylinder length=0.15 radius=0.02; visual cylinder length=0.15 radius=0.02
- link l_shoulder_tilt_link: mass 0.1 -> 0.01; geometry collision sphere radius=0.015; visual sphere radius=0.015
- link r_shoulder_pan_link: mass 0.02 -> 0.1; geometry collision cylinder length=0.15 radius=0.02; visual cylinder length=0.15 radius=0.02
- link r_shoulder_tilt_link: mass 0.1 -> 0.01; geometry collision sphere radius=0.015; visual sphere radius=0.015
Joints:
- added joint l_shoulder_roll_joint: type revolute, parent base_link, child l_shoulder_roll_link, origin xyz=0.0 0.12 0.10 rpy=0 0 0, axis 1 0 0, limit lower=-0.35 upper=2.36 effort=10 velocity=2.0
- added joint r_shoulder_roll_joint: type revolute, parent base_link, child r_shoulder_roll_link, origin xyz=0.0 -0.12 0.10 rpy=0 0 0, axis -1 0 0, limit lower=-0.35 upper=2.36 effort=10 velocity=2.0
- joint l_elbow_joint: parent l_shoulder_tilt_link -> l_shoulder_pan_link
- joint l_shoulder_pan_joint: origin xyz=0.0 0.12 0.10 rpy=0 0 0 -> xyz=0 0 0 rpy=0 0 0; parent base_link -> l_shoulder_tilt_link
- joint l_shoulder_tilt_joint: limit lower=-0.7854 upper=2.3562 effort=10 velocity=2.0 -> lower=-1.5708 upper=1.5708 effort=10 velocity=2.0; parent l_shoulder_pan_link -> l_shoulder_roll_link
- joint r_elbow_joint: parent r_shoulder_tilt_link -> r_shoulder_pan_link
- joint r_shoulder_pan_joint: origin xyz=0.0 -0.12 0.10 rpy=0 0 0 -> xyz=0 0 0 rpy=0 0 0; parent base_link -> r_shoulder_tilt_link
- joint r_shoulder_tilt_joint: limit lower=-0.7854 upper=2.3562 effort=10 velocity=2.0 -> lower=-1.5708 upper=1.5708 effort=10 velocity=2.0; parent r_shoulder_pan_link -> r_shoulder_roll_link

Commit message: fix archtecture

File: urdf/real_steel.urdf (robot description, URDF)
Before this commit: robot real_steel, 11 links, 10 joints
Links:
- removed link l_shoulder_roll_link
- removed link r_shoulder_roll_link
- added link torso_yaw_link, mass 0.05; collision cylinder length=0.02 radius=0.03; visual cylinder length=0.02 radius=0.03
- link l_shoulder_tilt_link: mass 0.01 -> 0.02; geometry collision sphere radius=0.025; visual sphere radius=0.025
- link r_shoulder_tilt_link: mass 0.01 -> 0.02; geometry collision sphere radius=0.025; visual sphere radius=0.025
Joints:
- removed joint l_shoulder_roll_joint
- removed joint r_shoulder_roll_joint
- added joint torso_yaw_joint: type revolute, parent base_link, child torso_yaw_link, origin xyz=0 0 0.125 rpy=0 0 0, axis 0 0 1, limit lower=-1.5708 upper=1.5708 effort=10 velocity=2.0
- joint l_shoulder_tilt_joint: origin xyz=0 0 0 rpy=0 0 0 -> xyz=0.0 0.12 0.10 rpy=0 0 0; parent l_shoulder_roll_link -> torso_yaw_link
- joint r_shoulder_tilt_joint: origin xyz=0 0 0 rpy=0 0 0 -> xyz=0.0 -0.12 0.10 rpy=0 0 0; parent r_shoulder_roll_link -> torso_yaw_link
